File: pcb/stm32pe_midi/stm32pe_midi.kicad_pcb (KiCad board)
At the start: 4 copper layers, 307 x 46.1 mm, 141 parts, among them J1 USB4105, J3 Conn_01x05_Pin, J4 Conn_01x10_Pin, J5 Conn_01x10_Socket, J6 Conn_01x05_Pin, SW1 SW_SPST, SW2 SW_SPST, U1 STM32H743VIHx, U10 TMAG5273, U11 TMAG5273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

Commit message: add wip firmware
Parts:
- removed mouse-bite-2mm-slot-1, mouse-bite-2mm-slot-2, mouse-bite-2mm-slot-3, mouse-bite-2mm-slot-4, mouse-bite-2mm-slot-5: VAL**, 1_udu_lib:mouse-bite-2mm-slot
Other:
- outline, holes or cut-outs redrawn
